File: simm-30-4mb.kicad_pcb (KiCad board)
At the start: 2 copper layers, 6 parts, among them J2 Conn_01x30, U1 511400, U2 511400

Commit message: more work
Parts:
- added C3: 100n, stdpads:C_1206, F.Cu at (176.0, 76.2)
- U1, U2: footprint stdpads:SOJ-24-26-300mil -> stdpads:SOP-24-26-300mil
- moved C3 12.8 mm to (159.5, 75.9)
- moved U1 12.7 mm to (148.7, 73.7)
- moved C1 1.32 mm to (103.6, 75.9)
- moved C2 1.32 mm to (125.2, 75.9)
Connections:
- U1 pad 2: /D7 -> /D5
- U1 pad 24: /D4 -> /D6
- U1 pad 25: /D6 -> /D4
- U1 pad 3: /D5 -> /D7
- U2 pad 2: /D0 -> /D1
- U2 pad 25: /D3 -> /D0
- U2 pad 3: /D1 -> /D3
Routing:
- net /~WE~: track 117.7 -> 20.0 mm, vias 4 -> 1
- net +5V: track 79.0 -> 0.00 mm
- net /1A5: track 44.8 -> 112.8 mm, vias 0 -> 2
- net /1A4: track 50.7 -> 114.1 mm, vias 0 -> 2
- net /~CASP~: track 0.00 -> 34.8 mm
- net /1A3: track 55.0 -> 20.9 mm, vias 0 -> 2
- net /~RAS~: track 110.5 -> 76.7 mm, vias 2 -> 1
- net /1A2: track 54.1 -> 21.5 mm, vias 0 -> 2
- net /D7: track 48.9 -> 24.4 mm, vias 1 -> 0
- net /D5: track 34.5 -> 13.4 mm, vias 1 -> 0
- net /1A9: track 62.8 -> 45.4 mm, vias 0 -> 2
- net /1A1: track 52.3 -> 68.5 mm, vias 0 -> 2
- net /1A6: track 47.6 -> 61.4 mm, vias 0 -> 2
- net /~CAS~: track 62.2 -> 48.7 mm, vias 3 -> 2
- net /1A10: track 61.3 -> 48.6 mm, vias 0 -> 2
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- removed copper zone on F.Cu, net +5V
Other:
- board outline added: 77.7 x 19 mm
- copper layers 2 -> 4
- net class Default: clearance 0.2 -> 0.127; trace_width 0.25 -> 0.127; via_dia 0.8 -> 0.508; via_drill 0.4 -> 0.2
- rule pad_to_mask_clearance: 0.2 -> 0.0762
- rule trace_clearance: 0.2 -> 0.127
- rule trace_min: 0.2 -> 0.127
- rule via_min_drill: 0.3 -> 0.2
- rule via_min_size: 0.4 -> 0.508
