File: simm-30-4mb.sch (KiCad schematic (older format))
At the start: 6 parts, among them J2 Conn_01x30, U1 511400, U2 511400

Commit message: more work
Connections:
- net D0: now also U2.25 (Pin_25); no longer U2.2 (Pin_2)
- net D1: now also U2.2 (Pin_2); no longer U2.3 (Pin_3)
- net D3: now also U2.3 (Pin_3); no longer U2.25 (Pin_25)
- net D4: now also U1.25 (Pin_25); no longer U1.24 (Pin_24)
- net D5: now also U1.2 (Pin_2); no longer U1.3 (Pin_3)
- net D6: now also U1.24 (Pin_24); no longer U1.25 (Pin_25)
- net D7: now also U1.3 (Pin_3); no longer U1.2 (Pin_2)
Changed lines of the file:
@@
 $EndComp
 Text Label 5500 4200 2    50   ~ 0
-D0
+D1
 Text Label 5500 4300 2    50   ~ 0
-D1
+D3
 Text Label 6000 4300 0    50   ~ 0
 D2
 Text Label 6000 4200 0    50   ~ 0
-D3
+D0
 Text Label 4100 4400 2    50   ~ 0
 ~WE~
@@
 $EndComp
 Text Label 4100 4200 2    50   ~ 0
+D5
+Text Label 4100 4300 2    50   ~ 0
 D7
-Text Label 4100 4300 2    50   ~ 0
-D5
 Text Label 4600 4300 0    50   ~ 0
+D6
+Text Label 4600 4200 0    50   ~ 0
 D4
-Text Label 4600 4200 0    50   ~ 0
-D6
 Text Label 5500 4400 2    50   ~ 0
 ~WE~
